File: CZ-6BM1.kicad_pcb (KiCad board)
At the start: 2 copper layers, 141 x 150 mm, 94 parts, among them IC1 74LS245, IC10 74LS393, IC11 74LS74, IC12 74ALS00, IC13 74LS00, IC14 74LS07, IC15 74LS157, IC16 NJM2903D, IC2 S260, IC3 74LS133, IC4 74LS08, IC5 74LS38, IC6 ym3802-x, IC7 74LS32, IC8 74LS04, IC9 74LS10, J1 x68000_expansion, J2 Mini-DIN-5 (out), J3 Mini-DIN-5 (through), J4 Mini-DIN-5 (IN), J5 Conn_Coaxial (sync in), J6 Conn_Coaxial (sync out), X1 16MHz, X2 4.9152MHz

Commit message: mk2
Parts:
- removed QR*****: cz-m1d1.flo.pe, cz-m1d1:cz-m1d1.flo.pe
- added ?: , , F.Cu at (116.5, 114.3)
- added ?: , , F.Cu at (129.3, 114.3)
- added ?: , , F.Cu at (110.5, 114.3)
- added REF**: DIP-16, CustomMountingHole:DIP-16, F.Cu at (126.7, 114.3)
- added REF**: DIP-16, CustomMountingHole:DIP-16, F.Cu at (108.0, 114.3)
- added TP10: TestPoint_Small, CustomMountingHole:TestPoint_THTPad_D1.0mm_Drill0.5mm, F.Cu at (134.8, 106.8)
- added TP11: TestPoint_Small, CustomMountingHole:TestPoint_THTPad_D1.0mm_Drill0.5mm, F.Cu at (142.2, 109.2)
- added TP12: TestPoint_Small, CustomMountingHole:TestPoint_THTPad_D1.0mm_Drill0.5mm, F.Cu at (134.8, 89.2)
- added TP13: TestPoint_Small, CustomMountingHole:TestPoint_THTPad_D1.0mm_Drill0.5mm, F.Cu at (134.8, 104.2)
- added TP14: TestPoint_Small, CustomMountingHole:TestPoint_THTPad_D1.0mm_Drill0.5mm, F.Cu at (142.2, 104.2)
- added TP15: TestPoint_Small, CustomMountingHole:TestPoint_THTPad_D1.0mm_Drill0.5mm, F.Cu at (134.8, 101.8)
- added TP16: TestPoint_Small, CustomMountingHole:TestPoint_THTPad_D1.0mm_Drill0.5mm, F.Cu at (142.2, 101.8)
- added TP17: TestPoint_Small, CustomMountingHole:TestPoint_THTPad_D1.0mm_Drill0.5mm, F.Cu at (137.2, 101.8)
- added TP18: TestPoint_Small, CustomMountingHole:TestPoint_THTPad_D1.0mm_Drill0.5mm, F.Cu at (137.2, 106.8)
- added TP19: TestPoint_Small, CustomMountingHole:TestPoint_THTPad_D1.0mm_Drill0.5mm, F.Cu at (139.8, 106.8)
- added TP20: TestPoint_Small, CustomMountingHole:TestPoint_THTPad_D1.0mm_Drill0.5mm, F.Cu at (137.2, 86.8)
- added TP21: TestPoint_Small, CustomMountingHole:TestPoint_THTPad_D1.0mm_Drill0.5mm, F.Cu at (137.2, 89.2)
- added TP22: TestPoint_Small, CustomMountingHole:TestPoint_THTPad_D1.0mm_Drill0.5mm, F.Cu at (134.8, 91.8)
- added TP23: TestPoint_Small, CustomMountingHole:TestPoint_THTPad_D1.0mm_Drill0.5mm, F.Cu at (134.8, 94.2)
- added TP24: TestPoint_Small, CustomMountingHole:TestPoint_THTPad_D1.0mm_Drill0.5mm, F.Cu at (134.8, 99.2)
- added TP25: TestPoint_Small, CustomMountingHole:TestPoint_THTPad_D1.0mm_Drill0.5mm, F.Cu at (137.2, 99.2)
- added TP26: TestPoint_Small, CustomMountingHole:TestPoint_THTPad_D1.0mm_Drill0.5mm, F.Cu at (139.8, 99.2)
- added TP27: TestPoint_Small, CustomMountingHole:TestPoint_THTPad_D1.0mm_Drill0.5mm, F.Cu at (142.2, 106.8)
- added TP28: TestPoint_Small, CustomMountingHole:TestPoint_THTPad_D1.0mm_Drill0.5mm, F.Cu at (139.8, 86.8)
- added TP29: TestPoint_Small, CustomMountingHole:TestPoint_THTPad_D1.0mm_Drill0.5mm, F.Cu at (139.8, 91.8)
- added TP30: TestPoint_Small, CustomMountingHole:TestPoint_THTPad_D1.0mm_Drill0.5mm, F.Cu at (137.2, 91.8)
- added TP31: TestPoint_Small, CustomMountingHole:TestPoint_THTPad_D1.0mm_Drill0.5mm, F.Cu at (142.2, 91.8)
- added TP32: TestPoint_Small, CustomMountingHole:TestPoint_THTPad_D1.0mm_Drill0.5mm, F.Cu at (134.8, 96.8)
- added TP33: TestPoint_Small, CustomMountingHole:TestPoint_THTPad_D1.0mm_Drill0.5mm, F.Cu at (137.2, 96.8)
- added TP34: TestPoint_Small, CustomMountingHole:TestPoint_THTPad_D1.0mm_Drill0.5mm, F.Cu at (142.2, 96.8)
- added TP35: TestPoint_Small, CustomMountingHole:TestPoint_THTPad_D1.0mm_Drill0.5mm, F.Cu at (139.8, 101.8)
- added TP36: TestPoint_Small, CustomMountingHole:TestPoint_THTPad_D1.0mm_Drill0.5mm, F.Cu at (142.2, 86.8)
- added TP37: TestPoint_Small, CustomMountingHole:TestPoint_THTPad_D1.0mm_Drill0.5mm, F.Cu at (139.8, 89.2)
- added TP38: TestPoint_Small, CustomMountingHole:TestPoint_THTPad_D1.0mm_Drill0.5mm, F.Cu at (142.2, 89.2)
- added TP39: TestPoint_Small, CustomMountingHole:TestPoint_THTPad_D1.0mm_Drill0.5mm, F.Cu at (137.2, 94.2)
- added TP4: TestPoint_Small, CustomMountingHole:TestPoint_THTPad_D1.0mm_Drill0.5mm, F.Cu at (134.8, 86.8)
- added TP40: TestPoint_Small, CustomMountingHole:TestPoint_THTPad_D1.0mm_Drill0.5mm, F.Cu at (142.2, 94.2)
- added TP41: TestPoint_Small, CustomMountingHole:TestPoint_THTPad_D1.0mm_Drill0.5mm, F.Cu at (139.8, 94.2)
- added TP42: TestPoint_Small, CustomMountingHole:TestPoint_THTPad_D1.0mm_Drill0.5mm, F.Cu at (139.8, 96.8)
- added TP43: TestPoint_Small, CustomMountingHole:TestPoint_THTPad_D1.0mm_Drill0.5mm, F.Cu at (142.2, 99.2)
- added TP44: TestPoint_Small, CustomMountingHole:TestPoint_THTPad_D1.0mm_Drill0.5mm, F.Cu at (134.8, 111.8)
- added TP45: TestPoint_Small, CustomMountingHole:TestPoint_THTPad_D1.0mm_Drill0.5mm, F.Cu at (116.5, 104.2)
- added TP45: TestPoint_Small, CustomMountingHole:TestPoint_THTPad_D1.0mm_Drill0.5mm, F.Cu at (97.8, 111.8)
- added TP45: TestPoint_Small, CustomMountingHole:TestPoint_THTPad_D1.0mm_Drill0.5mm, F.Cu at (110.5, 111.8)
- added TP45: TestPoint_Small, CustomMountingHole:TestPoint_THTPad_D1.0mm_Drill0.5mm, F.Cu at (129.3, 109.2)
- added TP45: TestPoint_Small, CustomMountingHole:TestPoint_THTPad_D1.0mm_Drill0.5mm, F.Cu at (110.5, 109.3)
- added TP45: TestPoint_Small, CustomMountingHole:TestPoint_THTPad_D1.0mm_Drill0.5mm, F.Cu at (129.3, 104.2)
- added TP45: TestPoint_Small, CustomMountingHole:TestPoint_THTPad_D1.0mm_Drill0.5mm, F.Cu at (116.5, 101.6)
- added TP45: TestPoint_Small, CustomMountingHole:TestPoint_THTPad_D1.0mm_Drill0.5mm, F.Cu at (110.5, 106.8)
- added TP45: TestPoint_Small, CustomMountingHole:TestPoint_THTPad_D1.0mm_Drill0.5mm, F.Cu at (129.2, 101.6)
- added TP45: TestPoint_Small, CustomMountingHole:TestPoint_THTPad_D1.0mm_Drill0.5mm, F.Cu at (116.5, 111.8)
- added TP45: TestPoint_Small, CustomMountingHole:TestPoint_THTPad_D1.0mm_Drill0.5mm, F.Cu at (129.3, 111.8)
- added TP45: TestPoint_Small, CustomMountingHole:TestPoint_THTPad_D1.0mm_Drill0.5mm, F.Cu at (129.2, 96.5)
- added TP45: TestPoint_Small, CustomMountingHole:TestPoint_THTPad_D1.0mm_Drill0.5mm, F.Cu at (116.5, 99.1)
- added TP45: TestPoint_Small, CustomMountingHole:TestPoint_THTPad_D1.0mm_Drill0.5mm, F.Cu at (110.5, 104.1)
- added TP45: TestPoint_Small, CustomMountingHole:TestPoint_THTPad_D1.0mm_Drill0.5mm, F.Cu at (110.5, 99.1)
- added TP45: TestPoint_Small, CustomMountingHole:TestPoint_THTPad_D1.0mm_Drill0.5mm, F.Cu at (134.8, 114.2)
- added TP45: TestPoint_Small, CustomMountingHole:TestPoint_THTPad_D1.0mm_Drill0.5mm, F.Cu at (97.8, 104.2)
- added TP45: TestPoint_Small, CustomMountingHole:TestPoint_THTPad_D1.0mm_Drill0.5mm, F.Cu at (97.8, 114.3)
- added TP45: TestPoint_Small, CustomMountingHole:TestPoint_THTPad_D1.0mm_Drill0.5mm, F.Cu at (116.5, 96.6)
- added TP45: TestPoint_Small, CustomMountingHole:TestPoint_THTPad_D1.0mm_Drill0.5mm, F.Cu at (116.5, 106.8)
- added TP45: TestPoint_Small, CustomMountingHole:TestPoint_THTPad_D1.0mm_Drill0.5mm, F.Cu at (97.8, 101.6)
- added TP45: TestPoint_Small, CustomMountingHole:TestPoint_THTPad_D1.0mm_Drill0.5mm, F.Cu at (110.5, 96.5)
- added TP45: TestPoint_Small, CustomMountingHole:TestPoint_THTPad_D1.0mm_Drill0.5mm, F.Cu at (97.8, 96.6)
- added TP45: TestPoint_Small, CustomMountingHole:TestPoint_THTPad_D1.0mm_Drill0.5mm, F.Cu at (129.2, 99.1)
- added TP45: TestPoint_Small, CustomMountingHole:TestPoint_THTPad_D1.0mm_Drill0.5mm, F.Cu at (116.5, 109.3)
- added TP45: TestPoint_Small, CustomMountingHole:TestPoint_THTPad_D1.0mm_Drill0.5mm, F.Cu at (97.8, 109.3)
- added TP45: TestPoint_Small, CustomMountingHole:TestPoint_THTPad_D1.0mm_Drill0.5mm, F.Cu at (97.8, 99.1)
- added TP45: TestPoint_Small, CustomMountingHole:TestPoint_THTPad_D1.0mm_Drill0.5mm, F.Cu at (110.5, 101.6)
- added TP45: TestPoint_Small, CustomMountingHole:TestPoint_THTPad_D1.0mm_Drill0.5mm, F.Cu at (97.8, 106.7)
- added TP45: TestPoint_Small, CustomMountingHole:TestPoint_THTPad_D1.0mm_Drill0.5mm, F.Cu at (129.3, 106.7)
- added TP46: TestPoint_Small, CustomMountingHole:TestPoint_THTPad_D1.0mm_Drill0.5mm, F.Cu at (137.2, 111.8)
- added TP47: TestPoint_Small, CustomMountingHole:TestPoint_THTPad_D1.0mm_Drill0.5mm, F.Cu at (137.2, 114.2)
- added TP48: TestPoint_Small, CustomMountingHole:TestPoint_THTPad_D1.0mm_Drill0.5mm, F.Cu at (139.8, 111.8)
- added TP49: TestPoint_Small, CustomMountingHole:TestPoint_THTPad_D1.0mm_Drill0.5mm, F.Cu at (139.8, 114.2)
- added TP5: TestPoint_Small, CustomMountingHole:TestPoint_THTPad_D1.0mm_Drill0.5mm, F.Cu at (134.8, 109.2)
- added TP50: TestPoint_Small, CustomMountingHole:TestPoint_THTPad_D1.0mm_Drill0.5mm, F.Cu at (142.2, 111.8)
- added TP51: TestPoint_Small, CustomMountingHole:TestPoint_THTPad_D1.0mm_Drill0.5mm, F.Cu at (142.2, 114.2)
- added TP52: TestPoint_Small, CustomMountingHole:TestPoint_THTPad_D1.0mm_Drill0.5mm, F.Cu at (132.2, 86.8)
- added TP53: TestPoint_Small, CustomMountingHole:TestPoint_THTPad_D1.0mm_Drill0.5mm, F.Cu at (132.2, 89.2)
- added TP54: TestPoint_Small, CustomMountingHole:TestPoint_THTPad_D1.0mm_Drill0.5mm, F.Cu at (132.2, 91.8)
- added TP55: TestPoint_Small, CustomMountingHole:TestPoint_THTPad_D1.0mm_Drill0.5mm, F.Cu at (95.6, 121.2)
- added TP56: TestPoint_Small, CustomMountingHole:TestPoint_THTPad_D1.0mm_Drill0.5mm, F.Cu at (95.6, 123.6)
- added TP57: TestPoint_Small, CustomMountingHole:TestPoint_THTPad_D1.0mm_Drill0.5mm, F.Cu at (95.6, 126.2)
- added TP58: TestPoint_Small, CustomMountingHole:TestPoint_THTPad_D1.0mm_Drill0.5mm, F.Cu at (95.6, 128.8)
- added TP59: TestPoint_Small, CustomMountingHole:TestPoint_THTPad_D1.0mm_Drill0.5mm, F.Cu at (95.6, 131.4)
- added TP6: TestPoint_Small, CustomMountingHole:TestPoint_THTPad_D1.0mm_Drill0.5mm, F.Cu at (137.2, 104.2)
- added TP60: TestPoint_Small, CustomMountingHole:TestPoint_THTPad_D1.0mm_Drill0.5mm, F.Cu at (95.6, 133.8)
- added TP61: TestPoint_Small, CustomMountingHole:TestPoint_THTPad_D1.0mm_Drill0.5mm, F.Cu at (95.6, 136.4)
- added TP62: TestPoint_Small, CustomMountingHole:TestPoint_THTPad_D1.0mm_Drill0.5mm, F.Cu at (95.6, 139.0)
- added TP7: TestPoint_Small, CustomMountingHole:TestPoint_THTPad_D1.0mm_Drill0.5mm, F.Cu at (139.8, 104.2)
- added TP8: TestPoint_Small, CustomMountingHole:TestPoint_THTPad_D1.0mm_Drill0.5mm, F.Cu at (137.2, 109.2)
- added TP9: TestPoint_Small, CustomMountingHole:TestPoint_THTPad_D1.0mm_Drill0.5mm, F.Cu at (139.8, 109.2)
- C10, C11, C12, C13, C14, C15, C16, C17, C18, C2, C21, C3, C4, C5, C6, C7, C8, C9: footprint Capacitor_THT:C_Rect_L7.0mm_W2.5mm_P5.00mm -> CustomMountingHole:C_Rect_L7.0mm_W2.5mm_P5.00mm_Custom
- X1, X2: footprint Crystal:Crystal_HC49-U_Horizontal_1EP_style2 -> CustomMountingHole:Crystal_HC49-U_Horizontal_1EP_style2_Custom
- moved J2 2.28 mm to (159.7, 100.0)
- moved J3 2.28 mm to (159.7, 117.6)
- moved J4 2.28 mm to (159.7, 135.4)
- moved J6 1.51 mm to (160.5, 83.0)
- moved J5 1.50 mm to (160.5, 68.1)
- moved C11 1.29 mm to (69.0, 85.3)
- moved R29 1.21 mm to (148.5, 137.4)
- moved PC1 1.04 mm to (148.4, 147.9)
- moved C8 0.76 mm to (51.3, 60.7)
- moved C6 0.72 mm to (51.1, 111.7)
- moved C9 0.72 mm to (74.0, 168.4)
- moved R28 0.69 mm to (140.8, 157.5)
- moved C5 0.66 mm to (51.4, 136.1)
- moved C21 0.64 mm to (121.9, 61.4)
- moved C7 0.62 mm to (51.2, 85.1)
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Routing:
- net GND: track 86.6 -> 1554.7 mm, vias 153 -> 9
- net +5V: track 844.6 -> 1126.9 mm, vias 2 -> 3
- net /4.0MHz: track 168.5 -> 207.0 mm, vias 1 -> 3
- net Net-(J2-Pad4): track 31.0 -> 51.7 mm, vias 0 -> 1
- net Net-(IC15-S): track 50.5 -> 67.7 mm, vias 0 -> 3
- net Net-(C20-Pad2): track 23.0 -> 38.8 mm
- net Net-(IC16-A_OUTPUT): track 136.3 -> 146.5 mm, vias 2 -> 1
- net Net-(J2-Pad5): track 54.5 -> 45.2 mm, vias 0 -> 1
- net Net-(IC12-Pad1): track 33.0 -> 23.8 mm
- net Net-(IC10A-CP): track 19.8 -> 27.7 mm, vias 0 -> 1
- net /AB1: track 180.5 -> 188.1 mm
- net Net-(IC11A-~{R}): track 90.6 -> 84.1 mm, vias 1 -> 2
- net Net-(IC11B-Q): track 42.9 -> 49.2 mm, vias 0 -> 2
- net Net-(IC6-CLICK): track 82.8 -> 88.7 mm
- net Net-(IC6-TxF): track 82.8 -> 88.7 mm
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Other:
- board text added: "10"
- board text added: "15"
- board text added: "20"
- board text added: "25"
- board text added: "30"
- board text added: "35"
- board text added: "40"
- board text added: "45"
- board text added: "5"
- board text added: "50"
- board text added: "A1"
- board text added: "JP1 1-2: ＄EAFA01～＄EAFA0F 2-3: ＄EAFA11～＄EAFA1F"
- board text added: "M1D1.FLO.PE 2"
- board text added: "SW1-1 On IRQ4 Off IRQ2"
- board text added: "SW1-2 On OUT Off THRU"
- board text added: "X68000"
- board text added: "ボード 1"
- board text added: "ボード 2"
- board text removed: "mk1"
